File: MINI-ULTRA-PRO.sch (KiCad schematic (older format))
At the start: 62 parts, among them J1 S2B-PH-SM4-TB, J2 MICRO-USB, J3 RF-SMA-EDGE, J4 CONN-HDR-1x19, J5 CONN-HDR-1x19, J6 CONN-HDR-2x5, M1 MOUNT_HOLE, M2 MOUNT_HOLE, M3 MOUNT_HOLE, M4 MOUNT_HOLE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

Commit message: Version 0.40
Parts:
- removed C18: 4.7nF 25V X7R, RocketScreamKicadLibrary:CAP-0402, symbol CAPACITOR-CERAMIC
- removed D2: LED-DUAL, RocketScreamKicadLibrary:LED-1615, symbol LED-DUAL
- removed D3: PRTR5V0U2X, RocketScreamKicadLibrary:SOT-143B, symbol PRTR5V0U2X
- removed J3: RF-SMA-EDGE, RocketScreamKicadLibrary:RF-SMA-EDGE, symbol RF-SMA-EDGE
- removed U4: MCP1700T-3302E/MB, RocketScreamKicadLibrary:SOT-89, symbol MCP1700T-XXX2E
- added C20: 100nF, RocketScreamKicadLibrary:C_0603, symbol CAPACITOR-CERAMIC
- added D2: Green, RocketScreamKicadLibrary:LED_0603, symbol LED-SINGLE
- added D3: Red, RocketScreamKicadLibrary:LED_0603, symbol LED-SINGLE
- added D5: PRTR5V0U2X, RocketScreamKicadLibrary:SOT-143B, symbol PRTR5V0U2X
- added J3: RF-SMA-EDGE_Without_Feed, RocketScreamKicadLibrary:RF-SMA-EDGE_Without_Feed, symbol RF-SMA-EDGE_Without_Feed
- added J7: U.FL-R-SMT, RocketScreamKicadLibrary:U.FL-R-SMT_Extended, symbol U.FL-R-SMT
- added J8: ANTENNA-PAD, RocketScreamKicadLibrary:ANTENNA-PAD, symbol ANTENNA-PAD
- added JP1, JP2, JP3: JUMPER-1-WAY, RocketScreamKicadLibrary:JUMPER-1-WAY-SMD, symbol JUMPER-1-WAY
- added L3: BLM18KG221SN1D, RocketScreamKicadLibrary:I_0603, symbol INDUCTOR
- added R14: 2K2, RocketScreamKicadLibrary:R_0603, symbol RESISTOR
- added U4: MCP1700T-3302E/MB, RocketScreamKicadLibrary:SOT-89, symbol MCP1700T-XXX2E/MB
- added U6: 24AA02E64T-I/OT, RocketScreamKicadLibrary:SOT-23-5, symbol 24AA02E64T-I/OT
- C1, C10, C12, C13, C14, C15, C16, C17, C19, C2, C3, C4, C5, C6, C7, C8: footprint RocketScreamKicadLibrary:CAP-0402 -> RocketScreamKicadLibrary:C_0603
- C11: value 4.7uF 10V X5R -> 47uF 10V X5R; footprint RocketScreamKicadLibrary:CAP-0402 -> RocketScreamKicadLibrary:C_0805
- C9: footprint RocketScreamKicadLibrary:CAP-0603 -> RocketScreamKicadLibrary:C_0603
- D1: value Orange -> Yellow; footprint RocketScreamKicadLibrary:LED-0603 -> RocketScreamKicadLibrary:LED_0603
- J6: footprint RocketScreamKicadLibrary:HDR_2x5_Pitch1.27mm -> RocketScreamKicadLibrary:HDR_2x5_Pitch1.27mm_SMD
- L1, L2: value BKP1005TS121-T -> BLM18KG221SN1D; footprint RocketScreamKicadLibrary:IND-0402 -> RocketScreamKicadLibrary:I_0603
- R1, R10, R11, R13, R2, R3, R4, R6, R7, R8, R9: footprint RocketScreamKicadLibrary:RES-0402 -> RocketScreamKicadLibrary:R_0603
- R12: value 10K -> 2K2; footprint RocketScreamKicadLibrary:RES-0402 -> RocketScreamKicadLibrary:R_0603
- R5: value 1M -> 2K2; footprint RocketScreamKicadLibrary:RES-0402 -> RocketScreamKicadLibrary:R_0603
Connections:
- wire segments 284 -> 309
- no-connect marks 16 -> 13
Other:
- note added: "1. All capacitors are NP0/COG 50V unless specified.\n2. All resistors are 62.5mW 1% unless specified.\n3. Close JP1, JP2, & JP3 to run LMIC stack."
- note added: "250mA"
- note added: "50Ohm"
- note added: "Close JP1, JP2 & JP3 \nto use Arduino-LMIC\nlibrary"
- note added: "EUI-64 MAC ID"
- note added: "Through hole pad\nfor 1/4 wave\nwire antenna"
- note removed: "1. All capacitors are NP0/COG 50V unless specified.\n2. All resistors are 62.5mW 1% unless specified."
- moved on the sheet: C11, C12, C13, U3, U5

Commit message: Version 0.50 - V3
Parts:
- added C18: 100nF, RocketScreamKicadLibrary:C_0603, symbol RocketScreamKicadLibrary:CAPACITOR-CERAMIC
- added LOGO4: LOGO-ROCKET-SCREAM, RocketScreamKicadLibrary:LOGO-ROCKET-SCREAM_Without_Text_XXXSmall, symbol RocketScreamKicadLibrary:LOGO-ROCKET-SCREAM
- added R15: 1M, RocketScreamKicadLibrary:R_0603, symbol RocketScreamKicadLibrary:RESISTOR
- added R16: 3M3, RocketScreamKicadLibrary:R_0603, symbol RocketScreamKicadLibrary:RESISTOR
- C1, C10, C11, C12, C13, C14, C15, C16, C17, C19, C2, C20, C3, C4, C5, C6, C7, C8, C9: symbol CAPACITOR-CERAMIC -> RocketScreamKicadLibrary:CAPACITOR-CERAMIC
- D1, D2, D3: symbol LED-SINGLE -> RocketScreamKicadLibrary:LED-SINGLE
- D4: symbol DIODE_DUAL_Schottky -> RocketScreamKicadLibrary:DIODE_DUAL_Schottky
- D5: symbol PRTR5V0U2X -> RocketScreamKicadLibrary:PRTR5V0U2X
- F1: symbol FUSE -> RocketScreamKicadLibrary:FUSE
- J1: symbol S2B-PH-SM4-TB -> RocketScreamKicadLibrary:S2B-PH-SM4-TB
- J2: symbol MICRO-USB -> RocketScreamKicadLibrary:MICRO-USB
- J3: symbol RF-SMA-EDGE_Without_Feed -> RocketScreamKicadLibrary:RF-SMA-EDGE_Without_Feed
- J4, J5: symbol CONN-HDR-1x19 -> RocketScreamKicadLibrary:CONN-HDR-1x19
- J6: symbol CONN-HDR-2x5 -> RocketScreamKicadLibrary:CONN-HDR-2x5
- J7: symbol U.FL-R-SMT -> RocketScreamKicadLibrary:U.FL-R-SMT
- J8: symbol ANTENNA-PAD -> RocketScreamKicadLibrary:ANTENNA-PAD
- JP1, JP2, JP3: symbol JUMPER-1-WAY -> RocketScreamKicadLibrary:JUMPER-1-WAY
- L1, L2, L3: symbol INDUCTOR -> RocketScreamKicadLibrary:INDUCTOR
- LOGO1: symbol LOGO-ROCKET-SCREAM -> RocketScreamKicadLibrary:LOGO-ROCKET-SCREAM
- LOGO2: symbol LOGO-OSHW -> RocketScreamKicadLibrary:LOGO-OSHW
- LOGO3: symbol LOGO-KICAD -> RocketScreamKicadLibrary:LOGO-KICAD
- M1, M2, M3, M4: symbol MOUNT_HOLE -> RocketScreamKicadLibrary:MOUNT_HOLE
- M5, M6: symbol FIDUCIAL -> RocketScreamKicadLibrary:FIDUCIAL
- Q1: symbol MOSFET-N -> RocketScreamKicadLibrary:MOSFET-N
- R1, R10, R11, R12, R13, R14, R2, R3, R4, R5, R6, R7, R8, R9: symbol RESISTOR -> RocketScreamKicadLibrary:RESISTOR
- SW1: symbol TACT-SWITCH_2Pins -> RocketScreamKicadLibrary:TACT-SWITCH_2Pins
- U1: symbol ATSAMD21G18A-AU -> RocketScreamKicadLibrary:ATSAMD21G18A-AU
- U2: symbol BQ24074 -> RocketScreamKicadLibrary:BQ24074
- U3: symbol RFM9xW -> RocketScreamKicadLibrary:RFM9xW
- U4: symbol MCP1700T-XXX2E/MB -> RocketScreamKicadLibrary:MCP1700T-XXX2E-MB
- U5: value S25FL116K0XMFI041 -> W25Q16JVSSIM; footprint RocketScreamKicadLibrary:SOIC-8-N -> RocketScreamKicadLibrary:SOIC-8-W; symbol S25FL1xxK0XM -> RocketScreamKicadLibrary:S25FL1xxK0XM
- U6: symbol 24AA02E64T-I/OT -> RocketScreamKicadLibrary:24AA02E64T-I-OT
- Y1: symbol CRYSTAL -> RocketScreamKicadLibrary:CRYSTAL
Connections:
- wire segments 309 -> 371
Other:
- note added: "BATTERY\nMONITORING"
- moved on the sheet: J6
